File: uaf0/TRANSISTOR_DI.sch (KiCad schematic (older format))
At the start: 10 parts

Commit message: откорректирована схема+добавлен тестовый скетч
Parts:
- R16, R17: Номинал 1 кОм -> 4,7 кОм; УГО R101 -> R472
Changed lines of the file:
@@
 F 2 "N_RLC:Резистор_SMD_0603_0,065_Вт" H 4800 2750 60  0001 C CNN
 F 3 "" H 4800 2750 60  0001 C CNN
-F 4 "R101" H 4800 2750 50  0001 C CNN "УГО"
-F 5 "1 кОм" H 4800 2600 50  0000 C CNN "Номинал"
+F 4 "R472" H 4800 2750 50  0001 C CNN "УГО"
+F 5 "4,7 кОм" H 4800 2600 50  0000 C CNN "Номинал"
 	1    4800 2750
 	1    0    0    -1
@@
 F 2 "N_RLC:Резистор_SMD_0603_0,065_Вт" H 4800 5250 60  0001 C CNN
 F 3 "" H 4800 5250 60  0001 C CNN
-F 4 "R101" H 4800 5250 50  0001 C CNN "УГО"
-F 5 "1 кОм" H 4800 5100 50  0000 C CNN "Номинал"
+F 4 "R472" H 4800 5250 50  0001 C CNN "УГО"
+F 5 "4,7 кОм" H 4800 5100 50  0000 C CNN "Номинал"
 	1    4800 5250
 	1    0    0    -1
